File: project/main.kicad_pcb (KiCad board)
At the start: 6 copper layers, 160 x 257 mm, 194 parts

Commit message: alternate placement for dirty workshop
Parts:
- removed R52: Trash el, -local:_o_trash_electronics__
- moved R19 149.5 mm to (83.0, 61.3), turned to 0 degrees
- moved R37 149.2 mm to (186.8, 176.3), turned to -90 degrees
- moved R18 144.2 mm to (89.8, 59.3), turned to 0 degrees
- moved R38 138.3 mm to (196.8, 176.3), turned to 180 degrees
- moved L43 129.8 mm to (95.3, 62.3)
- moved R49 125.5 mm to (88.3, 114.3)
- moved R25 118.3 mm to (141.3, 59.8), turned to 0 degrees
- moved R47 106.5 mm to (103.3, 116.8)
- moved R41 105.4 mm to (159.3, 152.8), turned to 0 degrees
- moved L40 94.1 mm to (186.3, 167.3), turned to 180 degrees
- moved R61 92.8 mm to (89.3, 82.6)
- moved R5 89.6 mm to (133.8, 59.8), turned to 0 degrees
- moved L14 84.9 mm to (96.3, 100.3)
- moved L17 84.9 mm to (96.3, 75.3)
- moved R40 76.0 mm to (197.3, 136.8), turned to 180 degrees
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Routing:
- net (no net): track 333.7 -> 331.1 mm
Other:
- board text added: "needs: * 1f 10A * air"
