File: project/main.kicad_sch (KiCad schematic)
At the start: 207 parts

Commit message: updating ventilation map
Parts:
- added R105: machine intake fan, -local:_q_laser_fan__, symbol Device:R
- added R106: heat exchanger, -local:_q_printers_fan__, symbol Device:R
- added R107: dirty big fan, -local:_q_paint_fan__, symbol Device:R
- R101: value Laser fan -> laser fan
- R102: value Paint fan -> dirty fan
- R103: value Printers fan -> air con
Other:
- moved on the sheet: Be1, Be2, Be3, Be4, Be5, Be6, Be7
